File: TryoutH401/KiCAD/Test1.kicad_sch (KiCad schematic)
At the start: 65 parts, among them J1 Conn_Coaxial_Small, P1 USB_C_Plug, Q1 Q_PNP_BCE, SW1 Reset Switch, U1 CH340N, U2 ESP32-PICO-D4, U4 DS1302Z+, U5 AT25SF081-SSHD-X, U6 MI6118, X1 Crystal, X3 Crystal

Commit message: Added newer files KiCAD and Pictures
Connections:
- net at BT1.1 (+), D19.1 (K), U4.5 (CE): no longer U2.42 (IO21)
Other:
- moved on the sheet: LED2, LED3, LED4, LED5, LED6, LED7
Changed lines of the file:
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@@
 	)
 	(junction
-		(at 224.79 -25.4)
-		(diameter 0)
-		(color 0 0 0 0)
-	)
-	(junction
 		(at 21.59 -21.59)
 		(diameter 0)
@@
 	(wire
 		(pts
-			(xy 224.79 -6.35) (xy 224.79 30.48)
-		)
-		(stroke
-			(width 0)
-			(type default)
-		)
-	)
-	(wire
-		(pts
 			(xy 19.05 -8.89) (xy 19.05 20.32)
 		)
@@
 	(wire
 		(pts
-			(xy 87.63 -24.13) (xy 90.17 -24.13)
+			(xy 314.96 26.67) (xy 314.96 118.11)
 		)
 		(stroke
@@
 	(wire
 		(pts
-			(xy 175.26 80.01) (xy 175.26 87.63)
+			(xy 87.63 -24.13) (xy 90.17 -24.13)
 		)
 		(stroke
@@
 	(wire
 		(pts
-			(xy 74.93 -5.08) (xy 78.74 -5.08)
+			(xy 175.26 80.01) (xy 175.26 87.63)
 		)
 		(stroke
@@
 	(wire
 		(pts
-			(xy 107.95 -15.24) (xy 104.14 -15.24)
+			(xy 74.93 -5.08) (xy 78.74 -5.08)
 		)
 		(stroke
@@
 	(wire
 		(pts
-			(xy 236.22 111.76) (xy 238.76 111.76)
+			(xy 107.95 -15.24) (xy 104.14 -15.24)
 		)
 		(stroke
@@
 	(wire
 		(pts
-			(xy 218.44 -25.4) (xy 224.79 -25.4)
+			(xy 236.22 111.76) (xy 238.76 111.76)
 		)
 		(stroke
@@
 	(wire
 		(pts
-			(xy 224.79 -6.35) (xy 218.44 -6.35)
-		)
-		(stroke
-			(width 0)
-			(type default)
-		)
-	)
-	(wire
-		(pts
 			(xy 251.46 -25.4) (xy 261.62 -25.4)
 		)
@@
 	(wire
 		(pts
+			(xy 224.79 26.67) (xy 314.96 26.67)
+		)
+		(stroke
+			(width 0)
+			(type default)
+		)
+	)
+	(wire
+		(pts
 			(xy 41.91 -11.43) (xy 45.72 -11.43)
 		)
@@
 	(wire
 		(pts
+			(xy 224.79 30.48) (xy 224.79 26.67)
+		)
+		(stroke
+			(width 0)
+			(type default)
+		)
+	)
+	(wire
+		(pts
 			(xy 107.95 -22.86) (xy 100.33 -22.86)
 		)
@@
 	(wire
 		(pts
+			(xy 289.56 118.11) (xy 314.96 118.11)
+		)
+		(stroke
+			(width 0)
+			(type default)
+		)
+	)
+	(wire
+		(pts
 			(xy 41.91 -16.51) (xy 35.56 -16.51)
 		)
@@
 	(wire
 		(pts
-			(xy 218.44 -6.35) (xy 218.44 -25.4)
-		)
-		(stroke
-			(width 0)
-			(type default)
-		)
-	)
-	(wire
-		(pts
 			(xy 209.55 30.48) (xy 209.55 2.54)
 		)
@@
 	(symbol
 		(lib_id "Device:LED")
-		(at 27.94 45.72 0)
+		(at 31.75 50.8 0)
 		(unit 1)
 		(exclude_from_sim no)
@@
 		(dnp no)
 		(property "Reference" "LED2"
-			(at 27.432 42.672 0)
+			(at 31.242 47.752 0)
 			(effects
 				(font
@@
 		)
 		(property "Value" "LED"
-			(at 26.3525 41.91 0)
+			(at 30.1625 46.99 0)
 			(effects
 				(font
@@
 		)
 		(property "Footprint" ""
-			(at 27.94 45.72 0)
+			(at 31.75 50.8 0)
 			(effects
 				(font
@@
 		)
 		(property "Datasheet" "~"
-			(at 27.94 45.72 0)
+			(at 31.75 50.8 0)
 			(effects
 				(font
@@
 		)
 		(property "Description" "Light emitting diode"
-			(at 27.94 45.72 0)
+			(at 31.75 50.8 0)
 			(effects
 				(font
@@
 	(symbol
 		(lib_id "Device:LED")
-		(at 39.37 45.72 0)
+		(at 46.99 50.8 0)
 		(unit 1)
 		(exclude_from_sim no)
@@
 		(dnp no)
 		(property "Reference" "LED3"
-			(at 38.608 42.672 0)
+			(at 46.228 47.752 0)
 			(effects
 				(font
@@
 		)
 		(property "Value" "LED"
-			(at 37.7825 41.91 0)
+			(at 45.4025 46.99 0)
 			(effects
 				(font
@@
 		)
 		(property "Footprint" ""
-			(at 39.37 45.72 0)
+			(at 46.99 50.8 0)
 			(effects
 				(font
@@
 		)
 		(property "Datasheet" "~"
-			(at 39.37 45.72 0)
+			(at 46.99 50.8 0)
 			(effects
 				(font
@@
 		)
 		(property "Description" "Light emitting diode"
-			(at 39.37 45.72 0)
+			(at 46.99 50.8 0)
 			(effects
 				(font
@@
 	(symbol
 		(lib_id "Device:LED")
-		(at 50.8 45.72 0)
+		(at 62.23 50.8 0)
 		(unit 1)
 		(exclude_from_sim no)
@@
 		(dnp no)
 		(property "Reference" "LED4"
-			(at 50.546 42.672 0)
+			(at 61.976 47.752 0)
 			(effects
 				(font
@@
 		)
 		(property "Value" "LED"
-			(at 49.2125 41.91 0)
+			(at 60.6425 46.99 0)
 			(effects
 				(font
@@
 		)
 		(property "Footprint" ""
-			(at 50.8 45.72 0)
+			(at 62.23 50.8 0)
 			(effects
 				(font
@@
 		)
 		(property "Datasheet" "~"
-			(at 50.8 45.72 0)
+			(at 62.23 50.8 0)
 			(effects
 				(font
@@
 		)
 		(property "Description" "Light emitting diode"
-			(at 50.8 45.72 0)
+			(at 62.23 50.8 0)
 			(effects
 				(font
@@
 	(symbol
 		(lib_id "Device:LED")
-		(at 62.23 45.72 0)
+		(at 77.47 50.8 0)
 		(unit 1)
 		(exclude_from_sim no)
@@
 		(dnp no)
 		(property "Reference" "LED5"
-			(at 61.468 41.91 0)
+			(at 76.708 46.99 0)
 			(effects
 				(font
@@
 		)
 		(property "Value" "LED"
-			(at 60.6425 41.91 0)
+			(at 75.8825 46.99 0)
 			(effects
 				(font
@@
 		)
 		(property "Footprint" ""
-			(at 62.23 45.72 0)
+			(at 77.47 50.8 0)
 			(effects
 				(font
@@
 		)
 		(property "Datasheet" "~"
-			(at 62.23 45.72 0)
+			(at 77.47 50.8 0)
 			(effects
 				(font
@@
 		)
 		(property "Description" "Light emitting diode"
-			(at 62.23 45.72 0)
+			(at 77.47 50.8 0)
 			(effects
 				(font
@@
 	(symbol
 		(lib_id "Device:LED")
-		(at 82.55 45.72 0)
+		(at 107.95 50.8 0)
 		(unit 1)
 		(exclude_from_sim no)
@@
 		(dnp no)
 		(property "Reference" "LED7"
-			(at 82.296 42.672 0)
+			(at 107.696 47.752 0)
 			(effects
 				(font
@@
 		)
 		(property "Value" "LED"
-			(at 80.9625 41.91 0)
+			(at 106.3625 46.99 0)
 			(effects
 				(font
@@
 		)
 		(property "Footprint" ""
-			(at 82.55 45.72 0)
+			(at 107.95 50.8 0)
 			(effects
 				(font
@@
 		)
 		(property "Datasheet" "~"
-			(at 82.55 45.72 0)
+			(at 107.95 50.8 0)
 			(effects
 				(font
@@
 		)
 		(property "Description" "Light emitting diode"
-			(at 82.55 45.72 0)
+			(at 107.95 50.8 0)
 			(effects
 				(font
@@
 	(symbol
 		(lib_id "Device:LED")
-		(at 72.39 45.72 0)
+		(at 92.71 50.8 0)
 		(unit 1)
 		(exclude_from_sim no)
@@
 		(dnp no)
 		(property "Reference" "LED6"
-			(at 71.882 42.418 0)
+			(at 92.202 47.498 0)
 			(effects
 				(font
@@
 		)
 		(property "Value" "LED"
-			(at 70.8025 41.91 0)
+			(at 91.1225 46.99 0)
 			(effects
 				(font
@@
 		)
 		(property "Footprint" ""
-			(at 72.39 45.72 0)
+			(at 92.71 50.8 0)
 			(effects
 				(font
@@
 		)
 		(property "Datasheet" "~"
-			(at 72.39 45.72 0)
+			(at 92.71 50.8 0)
 			(effects
 				(font
@@
 		)
 		(property "Description" "Light emitting diode"
-			(at 72.39 45.72 0)
+			(at 92.71 50.8 0)
 			(effects
 				(font
